File: hardware/electronique/cartographe/carte_avionique/01_energie_pm.kicad_sch (KiCad schematic)
At the start: 7 parts, among them J101 ENTREE RADIO / DOMAINE VOL, J103 ENTREE 6S CHARGE UTILE, J104 SORTIE CALCUL 12V, U101 PROTECTION A DEFINIR, U102 BLOC LM5146-Q1 CANDIDAT

Commit message: feat(hw): compléter CA01 et clarifier la synchronisation des captures
Parts:
- removed J101: ENTREE RADIO / DOMAINE VOL, symbol Connector_Generic:Conn_01x02
- added C101, C102: 220n / 100V, Capacitor_SMD:C_0603_1608Metric, symbol Device:C
- added C103: 220n / 50V; Ceff>=100n, Capacitor_SMD:C_0603_1608Metric, symbol Device:C
- added C104: 10n / 100V, Capacitor_SMD:C_0603_1608Metric, symbol Device:C
- added C105: 33u/100V EEE-FK2A330P, Capacitor_SMD:CP_Elec_8x10.5, symbol Device:C_Polarized
- added C110: 100n / 100V, Capacitor_SMD:C_0603_1608Metric, symbol Device:C
- added C111: 100n / 25V, Capacitor_SMD:C_0603_1608Metric, symbol Device:C
- added C112: 2u2 / 25V, Capacitor_SMD:C_0603_1608Metric, symbol Device:C
- added C113: 100n / 16V, Capacitor_SMD:C_0603_1608Metric, symbol Device:C
- added C114: 4n7 / 25V, Capacitor_SMD:C_0603_1608Metric, symbol Device:C
- added C115: 100p C0G / 50V, Capacitor_SMD:C_0603_1608Metric, symbol Device:C
- added C116: 1n C0G / 50V, Capacitor_SMD:C_0603_1608Metric, symbol Device:C
- added C117, C118, C119, C120, C121: 4u7/100V, Capacitor_SMD:C_1210_3225Metric, symbol Device:C
- added C122, C123, C124, C125, C126: 22u/25V, Capacitor_SMD:C_1210_3225Metric, symbol Device:C
- added L101: 6u8 XAL1010-682MED, Inductor_SMD:L_Coilcraft_XAL1010-XXX, symbol Device:L
- added Q101, Q102, Q103, Q104: CSD19531Q5A, Package_TO_SOT_SMD:TDSON-8-1, symbol Transistor_FET:CSD19531Q5A
- added R101, R103, R112: 100k 0.1%, Resistor_SMD:R_0603_1608Metric, symbol Device:R
- added R102: 8k06 0.1%, Resistor_SMD:R_0603_1608Metric, symbol Device:R
- added R104: 4k42 0.1%, Resistor_SMD:R_0603_1608Metric, symbol Device:R
- added R105: 100R, Resistor_SMD:R_0603_1608Metric, symbol Device:R
- added R110, R114: 2R2, Resistor_SMD:R_0603_1608Metric, symbol Device:R
- added R111: 24k9 1%, Resistor_SMD:R_0603_1608Metric, symbol Device:R
- added R113: 9k31 0.1%, Resistor_SMD:R_0603_1608Metric, symbol Device:R
- added R115: 750R 1%, Resistor_SMD:R_0603_1608Metric, symbol Device:R
- added R116: 10m 0.5% / 1W CAND., Resistor_SMD:R_2512_6332Metric, symbol Device:R
- added R117: 21k 0.1%, Resistor_SMD:R_0603_1608Metric, symbol Device:R
- added R118: 1k50 0.1%, Resistor_SMD:R_0603_1608Metric, symbol Device:R
- added R119: 8k06, Resistor_SMD:R_0603_1608Metric, symbol Device:R
- added R120: 51R1, Resistor_SMD:R_0603_1608Metric, symbol Device:R
- F101: value A_CALCULER -> 10A CAND. / DC-Icc?; Sizing_Status (none) -> À valider
- F102: value A_CALCULER -> 1A SF-0603F100-2 CAND.; footprint (none) -> Fuse:Fuse_0603_1608Metric; MPN (none) -> SF-0603F100-2; Sizing_Status (none) -> À valider
- J103: value ENTREE 6S CHARGE UTILE -> 6S W08 / XT30 CAND.; Sizing_Status (none) -> À valider
- J104: value SORTIE CALCUL 12V -> 12V_COMPUTE / XT30 CAND.; Sizing_Status (none) -> À valider
- U101: value PROTECTION A DEFINIR -> LM74800QDRRRQ1; footprint (none) -> Package_SON:WSON-12-1EP_3x3mm_P0.5mm_EP1.5x2.5mm; symbol CA01_Fonctions:Protection_amont_TBD -> CA01_Design:LM74800QDRRRQ1; MPN (none) -> LM74800QDRRRQ1; Sizing_Status (none) -> À valider; now in the parts list
- U102: value BLOC LM5146-Q1 CANDIDAT -> LM5146QRGYRQ1; footprint (none) -> Package_DFN_QFN:Texas_RGY_R-PVQFN-N20_EP2.05x3.05mm; symbol CA01_Fonctions:Buck_calcul_LM5146_TBD -> CA01_Design:LM5146QRGYRQ1; MPN (none) -> LM5146QRGYRQ1; Sizing_Status (none) -> À valider; now in the parts list
Connections:
- net 12V_COMPUTE: now also C122.1, C123.1, C124.1, C125.1, C126.1, L101.2, R117.1, R120.1; no longer U102.2 (OUT)
- net GND: now also U101.7 (GND), U102.12 (PGND), U102.15 (EP_GND), U102.21 (EP_GND), U102.6 (AGND), U102.8 (SYNCIN), C101.2, C102.2, C104.2, C105.2, C110.2, C112.2, C113.2, C117.2, C118.2, C119.2, C120.2, C121.2, C122.2, C123.2, C124.2, C125.2, C126.2, R102.2, R104.2, R111.2, R113.2, R116.2, R118.2; no longer U101.3 (GND), U102.3 (GND)
- net VIN_PAYLOAD_PROT: now also U101.9 (OUT), C105.1, C117.1, C118.1, C119.1, C120.1, C121.1, Q102.1 (S), Q102.2 (S), Q102.3 (S), Q103.5 (D), R110.1, R112.1; no longer U101.2 (OUT), U102.1 (IN)
- net 5V2_FLIGHT renamed 5V_AUX
- net VBAT_FUSED: no longer names the net of F101.2
- net VBAT_FUSED: now also U101.2 (A), U101.3 (VSNS), C101.1, Q101.1 (S), Q101.2 (S), Q101.3 (S), R101.1; no longer U101.1 (IN)
- new net: C111.2, L101.1, Q103.1 (S), Q103.2 (S), Q103.3 (S), Q104.5 (D), U102.19 (SW)
- new net: Q103.4 (G), U102.18 (HO)
- new net: C102.1, C103.2, Q101.5 (D), Q102.5 (D), U101.10 (VS), U101.12 (C)
- new net: Q102.4 (G), R105.1, U101.8 (HGATE)
- new net: C104.1, R105.2
- new net: C115.2, C116.2, R117.2, R118.1, R119.2, U102.5 (FB)
- new net: R112.2, R113.1, U102.1 (EN/UVLO)
- new net: R115.1, U102.11 (ILIM)
- new net: Q104.4 (G), U102.13 (LO)
- new net: C112.1, R114.2, U102.14 (VCC)
- new net: C111.1, R114.1, U102.17 (BST)
- new net: R111.1, U102.2 (RT)
- new net: C110.1, R110.2, U102.20 (VIN)
- new net: C113.1, U102.3 (SS/TRK)
- new net: C114.1, C115.1, U102.4 (COMP)
- new net: C116.1, R120.2
- new net: R101.2, R102.1, U101.6 (EN/UVLO)
- new net: R103.2, R104.1, U101.5 (OV)
- new net: Q104.1 (S), Q104.2 (S), Q104.3 (S), R115.2, R116.1
- new net: C103.1, U101.11 (CAP)
- new net: R103.1, U101.4 (SW)
- new net: C114.2, R119.1
- new net: Q101.4 (G), U101.1 (DGATE)
- no-connect marks 0 -> 5
Other:
- note added: "01 - Entree protegee et12V_COMPUTE | DIMENSIONNEMENT CANDIDAT / NON FABRICABLE"
- note added: "BUCK 12 V / 6 A — entrée à gauche, étage de puissance et sortie à droite"
- note added: "BUCK CALCUL CANDIDAT : 12 V / 6 A, 400 kHz ; VIN travail 18–25.2 V. Base TI EVM SNVU591 : compensation, Ceff et transitoires à revalider. Shunt 10m / 1W + ILIM 750R : valley 7.5A typ ; Kelvin obligatoire. Cout 5 x 22u : Ceff >= 60u à 12 V à justifier. L6u8 : saturation/thermique ; EN 14.09/13.09 V. PCB/DRC, SOA et banc non qualifiés."
- note added: "FB / COMP : diviseur, avance de phase et compensation regroupés"
- note added: "PM08-CAN/PDB hors CA01 : BEC1->POWER1 ; BEC2->POWER2. CA01 ne porte pas la propulsion. F101 : protection W08 proche PDB a fermer. CANDIDATS : UV 16.50/15.18V ; OV 29.08/26.70V (recup. min25.70V), pas seuil batterie PX4. TVS NON SELECTEE ; transitoires/energie/SOA, Icc et appel charge a valider. LM74800 n'est pas une limitation de surcourant. RTN13 reste FLOTTANT."
- note added: "PWR_FLAG : sources physiques 6S/GND, nœuds après F101/FETs et filtre VIN. Aucun flag ne prouve protections ou dimensionnement."
- note removed: "01_energie_pm - ETUDE / NON FABRICABLE"
- note removed: "BLOC FONCTIONNEL seulement : FET, inductance, compensation, feedback et protections calcul/Jetson NON DESSINES."
- note removed: "CA01 EXCLUT LE COURANT PROPULSION. GND commun : pas d isolation galvanique. Selectivite a demontrer."
- note removed: "PM02D SUR SUPPORT SEPARE PM -> PIXHAWK POWER1 DIRECT, HORS CA01 Pas de transit 5V vol / I2C Pixhawk sur CA01. J101 = depart radio seul, protege en amont. Derivation externe et budget 5V2 a definir."
- note removed: "PM02D complet en tete batterie -> distribution. Faisceau adapte ; BEC vol conserve, POWER1 direct. Mesure globale via PM : calibration a valider."
- moved on the sheet: F101, F102, J103, J104
