File: hardware/electronique/cartographe/carte_avionique/05_synchronisation.kicad_sch (KiCad schematic)
At the start: 12 parts, among them J501 ADAPTATEUR AIRY SYNC, J502 BASLER M8-6 LOGIQUE, Q501 MMBT3904 CAND., U501 NIVEAU AIRY INCONNU, U502 SN74LVC1G17 CAND., U503 REGULATEUR A DEFINIR

Commit message: feat(hw): compléter CA01 et clarifier la synchronisation des captures
Parts:
- removed J501: ADAPTATEUR AIRY SYNC, symbol Connector_Generic:Conn_01x02
- removed J502: BASLER M8-6 LOGIQUE, symbol Connector_Generic:Conn_01x06
- removed JP501: OUVERT / NE PAS PONTER, symbol Jumper:Jumper_2_Open
- removed Q501: MMBT3904 CAND., Package_TO_SOT_SMD:SOT-23, symbol Transistor_BJT:MMBT3904
- removed R501: 1k CAND., symbol Device:R
- removed R502: 47k CAND., symbol Device:R
- removed R503: 100k CAND., symbol Device:R
- removed U501: NIVEAU AIRY INCONNU, symbol CA01_Fonctions:Adaptation_Airy_TBD
- removed U502: SN74LVC1G17 CAND., symbol 74xGxx:74LVC1G17
- removed U503: REGULATEUR A DEFINIR, symbol CA01_Fonctions:Regulateur_3V3_TBD
- added C502: 4.7uF / 10V X7R, Capacitor_SMD:C_0805_2012Metric, symbol Device:C
- added C503: 100nF / 10V, Capacitor_SMD:C_0603_1608Metric, symbol Device:C
- added C504, C505, C506, C507, C508, C509, C510, C511, C512, C513, C521: 100nF / 25V X7R, Capacitor_SMD:C_0603_1608Metric, symbol Device:C
- added C514, C515: 10uF / 25V X7R, Capacitor_SMD:C_1206_3216Metric, symbol Device:C
- added C516, C517, C518, C519: 1uF / 25V X7R, Capacitor_SMD:C_0805_2012Metric, symbol Device:C
- added C520: 2.2uF / 25V X7R, Capacitor_SMD:C_0805_2012Metric, symbol Device:C
- added D501: BAT54H, Diode_SMD:D_SOD-123F, symbol Device:D_Schottky
- added D502: BZT52H-C4V7, Diode_SMD:D_SOD-123F, symbol Device:D_Zener
- added D503, D504: TPD1E05U06DPYR, Package_SON:Texas_DPY0002A_0.6x1mm_P0.65mm, symbol CA01_Design:TPD1E05U06DPYR
- added J501: AIRY_SYNC_OUT1_W17_DNP, symbol CA01_Fonctions:Conn_01x02_LOGIQUE
- added J502: BASLER_M8_6_W18_W34, symbol CA01_Fonctions:Conn_01x06_LOGIQUE
- added J503: GNSS_G4_UART2_W36, symbol CA01_Fonctions:Conn_01x06_LOGIQUE
- added J504: AIRY_TEMPS_W23, symbol CA01_Fonctions:Conn_01x04_LOGIQUE
- added J505: ORIN_GPIO_PPS_W24, symbol CA01_Fonctions:Conn_01x02_LOGIQUE
- added J506: ORIN_DEBUG_GPRMC_W24, symbol CA01_Fonctions:Conn_01x02_LOGIQUE
- added J507: PIXHAWK_AUX1_W33, symbol CA01_Fonctions:Conn_01x02_LOGIQUE
- added J508: PIXHAWK_CAP1_W35, symbol CA01_Fonctions:Conn_01x02_LOGIQUE
- added J509: ORIN_CSI22_3V3_REF, symbol CA01_Fonctions:Conn_01x02_LOGIQUE
- added JP501: OUVERT_DNP, symbol CA01_Fonctions:Jumper_2_Open_DNP
- added Q501: PMV30UN2, Package_TO_SOT_SMD:SOT-23, symbol Transistor_FET:Q_NMOS_GSD
- added R510, R534, R535: 330R / 1%, Resistor_SMD:R_0603_1608Metric, symbol Device:R
- added R511, R543: 100k / 1%, Resistor_SMD:R_0603_1608Metric, symbol Device:R
- added R512: 4.7k / 0.25W, Resistor_SMD:R_1206_3216Metric, symbol Device:R
- added R513, R514: 1k / 1%, Resistor_SMD:R_0603_1608Metric, symbol Device:R
- added R530, R531: 47R / 1% DNP, Resistor_SMD:R_0603_1608Metric, symbol Device:R
- added R532, R533: 100R / 1% DNP, Resistor_SMD:R_0603_1608Metric, symbol Device:R
- added R536, R537: 22k / 1%, Resistor_SMD:R_0603_1608Metric, symbol Device:R
- added R538, R539: 3.01k / 1%, Resistor_SMD:R_0603_1608Metric, symbol Device:R
- added R540: 10k / 1%, Resistor_SMD:R_0603_1608Metric, symbol Device:R
- added R541, R542: 47k / 1%, Resistor_SMD:R_0603_1608Metric, symbol Device:R
- added U503: TPS7A2033PDBVR, Package_TO_SOT_SMD:SOT-23-5, symbol Regulator_Linear:TPS7A20xxxDBV
- added U504, U505, U507, U511: SN74LVC1T45DBVR, Package_TO_SOT_SMD:SOT-23-6, symbol CA01_Design:SN74LVC1T45DBVR
- added U506: TRS3232EIDR, Package_SO:SOIC-16_3.9x9.9mm_P1.27mm, symbol CA01_Design:TRS3232EIDR
- added U509: SN74LVC1G17DBVR, Package_TO_SOT_SMD:SOT-23-5, symbol 74xGxx:74LVC1G17
- added U510: TPS70950DBVR, Package_TO_SOT_SMD:SOT-23-5, symbol CA01_Design:TPS70950DBVR
- added U512, U513: SN74LVC1G17DBVR, Package_TO_SOT_SMD:SOT-23-5, symbol CA01_Design:SN74LVC1G17DBVR
- C501: value 100n / 10V CAND. -> 4.7uF / 10V X7R; footprint (none) -> Capacitor_SMD:C_0805_2012Metric
- F501: value A_CALCULER -> 400mA / SF-0603F040-2; footprint (none) -> Fuse:Fuse_0603_1608Metric
Connections:
- net 3V3_SYNC: now also C502.1, C503.1, C504.1, C506.1, C508.1, C510.1, C512.1, C513.1, R538.1, U503.5 (OUT), U504.1 (VCCA), U504.5 (DIR), U505.1 (VCCA), U505.5 (DIR), U507.1 (VCCA), U507.5 (DIR), U509.5 (VCC), U511.1 (VCCA), U511.5 (DIR), U512.5 (VCC), U513.5 (VCC); no longer C501.1
- net 5V_SYNC: now also C501.1, D501.2 (A), J502.2 (Pin_2), U503.1 (IN), U503.3 (EN)
- net AIRY_SYNC_RAW: now also J501.1 (Pin_1), JP501.1
- net BASLER_OPTO_RETURN: now also J502.3 (Pin_3), Q501.3 (D)
- net GND: now also C502.2, C503.2, C504.2, C505.2, C506.2, C507.2, C508.2, C509.2, C510.2, C511.2, C512.2, C513.2, C514.2, C515.2, C518.2, C519.2, C520.2, C521.2, D502.2 (A), D503.2 (GND), D504.2 (GND), J501.2 (Pin_2), J502.6 (Pin_6), J503.6 (Pin_6), J504.3 (Pin_3), J504.4 (Pin_4), J505.2 (Pin_2), J506.2 (Pin_2), J507.2 (Pin_2), J508.2 (Pin_2), J509.2 (Pin_2), Q501.2 (S), R511.2, R536.2, R537.2, R538.2, R539.2, R540.2, R541.2, R542.2, U503.2 (GND), U504.2 (GND), U505.2 (GND), U506.15 (GND), U507.2 (GND), U509.3 (GND), U510.2 (GND), U511.2 (GND), U512.3 (GND), U513.3 (GND)
- new net: R514.2, U509.4
- new net: C519.1, U506.6 (V-)
- new net: D502.1 (K), R512.1, U509.2
- new net: Q501.1 (G), R510.1, R511.1
- new net: R532.2, U505.4 (B)
- new net: C516.1, U506.1 (C1+)
- new net: R531.2, U506.14 (DOUT1)
- new net: C518.1, U506.2 (V+)
- new net: C516.2, U506.3 (C1-)
- new net: C517.1, U506.4 (C2+)
- new net: C517.2, U506.5 (C2-)
- new net: R530.2, U504.4 (B)
- new net: R533.2, U507.4 (B)
- new net: R535.1, R537.1, U513.2 (A)
- new net: D501.1 (K), R513.1
- new net: R534.1, R536.1, U512.2 (A)
- new net 12V_LIDAR: C514.1, U510.1 (IN)
- new net 3V3_ORIN_IO_REF: C505.1, C507.1, J509.1 (Pin_1), R540.1, U505.6 (VCCB), U507.6 (VCCB)
- new net 5V_AIRY_IO: C509.1, C511.1, C515.1, C520.1, C521.1, R539.1, R543.1, U504.6 (VCCB), U506.10 (DIN2), U506.16 (VCC), U510.5 (OUT), U511.6 (VCCB)
- new net AIRY_UART_LOGIC: R543.2, U506.11 (DIN1), U511.4 (B)
- new net BASLER_EXPOSURE_RAW: J502.4 (Pin_4), R512.2, R513.2
- new net FCU_AUX1: J507.1 (Pin_1), R510.2
- new net FCU_CAP1: J508.1 (Pin_1), R514.1
- new net GNSS_GPRMC_BUFFERED: U507.3 (A), U511.3 (A), U513.4 (Y)
- new net GNSS_GPRMC_IN: D504.1 (IO), J503.3 (Pin_3), R535.2
- new net GNSS_PPS_BUFFERED: U504.3 (A), U505.3 (A), U512.4 (Y)
- new net GNSS_PPS_IN: D503.1 (IO), J503.5 (Pin_5), R534.2
- new net GPRMC_AIRY: J504.2 (Pin_2), R531.1
- new net GPRMC_ORIN: J506.1 (Pin_1), R533.1, R542.1
- new net PPS_AIRY: J504.1 (Pin_1), R530.1
- new net PPS_ORIN: J505.1 (Pin_1), R532.1, R541.1
- no-connect marks 5 -> 17
Other:
- note added: "05 - SYNCHRONISATION / CIRCUITS CANDIDATS - NON FABRICABLE"
- note added: "3V3 : budget 50mA ; P LDO <=0.100W a 5.25V. CIN/COUT : Ceff >=0.47uF a verifier sous polarisation. F501 : budget total 5V_SYNC 80mA, protection secondaire 400mA candidate ; appel, chaud et selectivite a verifier."
- note added: "AIRY : rail IO lie au 12V LiDAR et conversion RS232 candidate"
- note added: "ALIMENTATION 3V3 LOCALE"
- note added: "BROCHAGES FABRICANTS REPRESENTES ; CIRCUITS CANDIDATS / NON FABRICABLE"
- note added: "CAMERA : AUX1 -> opto Line1 ; ExposureActive -> CAP1"
- note added: "JP501/2 NC : aucun lien vers la commande camera."
- note added: "Line1 : >5mA requis, <15mA limite en interne. Q501 gate 330R / rappel100k ; retour opto distinct de GND GPIO. M8 pin2 Line1, pin3 retour commute ; pin4 Line2, pin6 GND. Pins1/5 NC ; camera alimentee par USB3 externe."
- note added: "Line2 : rappel 5V via diode ; tampon3V3 tolere 5.5V/Ioff. R512 + D502 : protection DC candidate, pas qualification ESD. 24V : I~4.1mA, P R~80mW ; fronts et temperature a mesurer. Pixhawk/Orin eteints avec CA01 active : injection reste a verifier. CAP1 reserve a exposition, aucun PPS ; polarite/FrameID a valider."
- note added: "OPTION AIRY SYNC_OUT1 : OUVERTE / DNP"
- note added: "PPS + RMC GNSS : niveaux source, date et fronts a mesurer. R530-R533 DNP : banc requis avant raccordement cibles. RS232 Airy candidat exclusif ; adaptation TTL a revoir si besoin. 3V3_SYNC/Orin/Airy : sequence, fuites et charges a qualifier. Aucun ordre photo par PPS ; Jetson decide, PX4 declenche."
- note added: "REFERENCE ORIN : J509/1 = CSI22 VDD3.3 J509/2 = CSI GND1 ; retour requis pour isolation. GPIO/debug ne fournissent pas cette reference."
- note added: "TEMPS GNSS : entree protegee et Schmitt, sorties vers Orin"
- note added: "U510 EN ouvert : activation interne TPS709 ; NC4 ouvert. Ceff LDO >=2.2uF ; pompe TRS : valeurs sous biais a confirmer."
- note removed: "05_synchronisation - ETUDE / NON FABRICABLE"
- note removed: "R503 : rappel entree buffer au repos ; 100k candidat a valider."
- note removed: "SYNC_OUT1 Airy pin10 / fil D2 ; retour D4 : faisceau exact a verifier. Amplitude / courant inconnus : adaptation U501 non definie, JP501 ouvert. Basler pin2 Line1 ; pin3 retour opto COMMUTE (ne pas relier a GND). USB alimente la camera ; pas d isolation systeme garantie."
